Commit message: Updated URDF and matlab models

File: threelink_description/urdf/threelink.xacro (robot description, xacro)
@@ -1,4 +1,4 @@
 <?xml version="1.0"?>
-<!-- UNIMATE Puma 560 Manipulator -->
+<!-- Threelink model -->
 <robot name="threelink" xmlns:xacro="http://www.ros.org/wiki/xacro">
   <!-- Some constants -->
@@ -75,5 +75,5 @@
           <parent link="world"/>
           <child link="link_1"/>
-          <origin xyz="0 0 ${2 * length}" rpy="0 0 0" />
+          <origin xyz="0 0 ${3 * length}" rpy="0 0 0" />
           <axis xyz="1 0 0" />
           <dynamics damping="50.0"/>
@@ -87,5 +87,8 @@
           <origin xyz="0 0 ${- length}" rpy="0 0 0" />
           <axis xyz="1 0 0" />
-          <dynamics damping="50.0" spring_stiffness="200.0" />
+          <dynamics damping="50.0"/>
+          <dynamics friction="0.0"/>
+          <dynamics spring_reference="0.0"/>
+          <dynamics spring_stiffness="10.0"/>
         </joint>
         <joint name="joint_3" type="continuous">
@@ -94,5 +97,8 @@
           <origin xyz="0 0 ${- length}" rpy="0 0 0" />
           <axis xyz="1 0 0" />
-          <dynamics damping="50.0" spring_stiffness="200.0" />
+          <dynamics damping="50.0"/>
+          <dynamics friction="0.0"/>
+          <dynamics spring_reference="0.0"/>
+          <dynamics spring_stiffness="10.0"/>
         </joint>
         <transmission name="joint_1_transmission">
